File: split-keyboard-40/split-keyboard-40.kicad_pcb (KiCad board)
At the start: 2 copper layers, 85 parts, among them SW1 Switch, SW10 Switch, SW11 Switch, SW12 Switch, SW13 Switch, SW14 Switch, SW15 Switch, SW16 Switch, SW17 Switch, SW18 Switch, SW19 Switch, SW2 Switch, SW20 Switch, SW21 Switch, SW22 Switch, SW23 Switch, SW24 Switch, SW25 Switch, SW26 Switch, SW27 Switch, SW28 Switch, SW29 Switch, SW3 Switch, SW30 Switch, SW31 Switch, SW32 Switch, SW33 Switch, SW34 Switch, SW35 Switch, SW36 Switch, SW37 Switch, SW38 Switch, SW39 Switch, SW4 Switch, SW40 Switch, SW41 Switch, SW42 Switch, SW5 Switch, SW6 Switch, SW7 Switch, SW8 Switch, SW9 Switch, U1 Raspberry_Pi_Pico

Commit message: basic routing
Parts:
- D1, D10, D11, D12, D13, D14, D15, D16, D17, D18, D19, D2, D20, D21, D22, D23, D24, D25, D26, D27, D28, D29, D3, D30, D31, D32, D33, D34, D35, D36, D37, D38, D39, D4, D40, D41, D42, D5, D6, D7, D8, D9: moved to B.Cu
- moved D34 217.1 mm to (269.3, 56.1), turned to 105 degrees
- moved D35 215.8 mm to (274.3, 74.5), turned to 105 degrees
- moved D36 215.5 mm to (279.2, 92.9), turned to 105 degrees
- moved D31 194.6 mm to (250.3, 58.6), turned to 105 degrees
- moved D33 193.8 mm to (260.2, 95.4), turned to 105 degrees
- moved D32 193.5 mm to (255.3, 77.3), turned to 105 degrees
- moved D28 172.6 mm to (230.4, 58.0), turned to 105 degrees
- moved D30 172.2 mm to (240.3, 94.8), turned to 105 degrees
- moved D29 171.6 mm to (235.3, 76.4), turned to 105 degrees
- moved D25 168.8 mm to (211.5, 61.1), turned to 105 degrees
- moved D26 165.9 mm to (216.4, 79.5), turned to 105 degrees
- moved D27 164.6 mm to (221.4, 97.9), turned to 105 degrees
- moved D42 147.1 mm to (223.8, 121.5), turned to 105 degrees
- moved D22 144.4 mm to (194.1, 69.7), turned to 105 degrees
- moved SW16 143.3 mm to (80.7, 100.3), turned to -15 degrees
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Routing:
- net row_2: track 0.00 -> 235.6 mm
- net row_1: track 0.00 -> 232.8 mm
- net row_3: track 0.00 -> 232.8 mm
- net row_4: track 0.00 -> 204.3 mm
- net col_4: track 0.00 -> 135.6 mm, vias 0 -> 7
- net col_5: track 0.00 -> 116.3 mm, vias 0 -> 7
- net col_6: track 0.00 -> 106.6 mm, vias 0 -> 6
- net col_7: track 0.00 -> 76.2 mm
- net col_8: track 0.00 -> 68.3 mm, vias 0 -> 6
- net col_9: track 0.00 -> 66.7 mm, vias 0 -> 6
- net col_3: track 0.00 -> 38.1 mm, vias 0 -> 4
- net col_2: track 0.00 -> 38.1 mm, vias 0 -> 4
- net col_12: track 0.00 -> 38.1 mm, vias 0 -> 4
- net col_11: track 0.00 -> 38.1 mm, vias 0 -> 4
- net col_10: track 0.00 -> 38.1 mm, vias 0 -> 4
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
Commit message: keyboard layout
Parts:
- moved U1 152.4 mm to (149.2, -39.4)
- moved D34 19.7 mm to (283.0, 70.3), turned to 90 degrees
- moved D37 19.2 mm to (138.5, 134.9), turned to 70 degrees
- moved SW34 18.0 mm to (274.3, 69.7), turned to 0 degrees
- moved D6 17.2 mm to (127.4, 66.1), turned to 90 degrees
- moved D35 17.2 mm to (283.0, 89.3), turned to 90 degrees
- moved SW19 17.1 mm to (179.1, 65.9), turned to 0 degrees
- moved SW37 17.0 mm to (129.0, 134.9), turned to -20 degrees
- moved D31 16.5 mm to (264.0, 67.8), turned to 90 degrees
- moved D36 16.0 mm to (283.0, 108.4), turned to 90 degrees
- moved SW1 15.6 mm to (22.7, 69.6), turned to 0 degrees
- moved D19 15.6 mm to (187.8, 66.5), turned to 90 degrees
- moved SW6 15.3 mm to (117.9, 65.8), turned to 0 degrees
- moved SW35 15.2 mm to (274.3, 88.7), turned to 0 degrees
- moved SW31 15.1 mm to (255.3, 67.8), turned to 0 degrees
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Routing:
- net col_4: track 135.6 -> 0.00 mm, vias 7 -> 0
- net col_5: track 116.3 -> 1.95 mm, vias 7 -> 0
- net col_6: track 106.6 -> 0.00 mm, vias 6 -> 0
- net row_4: track 204.3 -> 123.0 mm
- net col_8: track 68.3 -> 0.00 mm, vias 6 -> 0
- net col_9: track 66.7 -> 0.00 mm, vias 6 -> 0
- net col_3: track 38.1 -> 0.00 mm, vias 4 -> 0
- net col_2: track 38.1 -> 0.00 mm, vias 4 -> 0
- net col_11: track 38.1 -> 0.00 mm, vias 4 -> 0
- net col_10: track 38.1 -> 0.00 mm, vias 4 -> 0
- net col_12: track 38.1 -> 0.03 mm, vias 4 -> 0

Commit message: routing of both sides, rotation
Parts:
- moved U1 170.4 mm to (149.2, 131.1)
- moved D34 26.8 mm to (265.0, 50.4), turned to 110 degrees
- moved SW1 25.2 mm to (41.5, 52.8), turned to -20 degrees
- moved SW34 24.4 mm to (256.6, 52.9), turned to 20 degrees
- moved D35 24.0 mm to (271.5, 68.3), turned to 110 degrees
- moved D6 23.6 mm to (141.1, 85.3), turned to 70 degrees
- moved D1 22.7 mm to (50.5, 55.9), turned to 70 degrees
- moved D36 22.7 mm to (278.0, 86.2), turned to 110 degrees
- moved D31 22.1 mm to (246.2, 54.6), turned to 110 degrees
- moved SW7 21.8 mm to (34.9, 70.7), turned to -20 degrees
- moved D37 21.6 mm to (128.0, 153.8), turned to 50 degrees
- moved SW6 21.5 mm to (132.3, 81.8), turned to -20 degrees
- moved SW35 21.2 mm to (263.1, 70.8), turned to 20 degrees
- moved SW2 20.9 mm to (60.0, 57.5), turned to -20 degrees
- moved SW19 20.8 mm to (165.8, 81.9), turned to 20 degrees
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Connections:
- U1 pad 1: row_1 -> col_1
- U1 pad 10: col_5 -> row_2
- U1 pad 11: col_6 -> row_3
- U1 pad 12: col_7 -> unconnected-(U1-GPIO9-Pad12)
- U1 pad 14: col_8 -> unconnected-(U1-GPIO10-Pad14)
- U1 pad 15: col_9 -> unconnected-(U1-GPIO11-Pad15)
- U1 pad 16: col_10 -> unconnected-(U1-GPIO12-Pad16)
- U1 pad 17: col_11 -> unconnected-(U1-GPIO13-Pad17)
- U1 pad 19: col_12 -> unconnected-(U1-GPIO14-Pad19)
- U1 pad 2: row_2 -> col_2
- U1 pad 22: unconnected-(U1-GPIO17-Pad22) -> col_7
- U1 pad 24: unconnected-(U1-GPIO18-Pad24) -> col_8
- U1 pad 25: unconnected-(U1-GPIO19-Pad25) -> col_9
- U1 pad 26: unconnected-(U1-GPIO20-Pad26) -> col_10
- U1 pad 27: unconnected-(U1-GPIO21-Pad27) -> col_11
- U1 pad 29: unconnected-(U1-GPIO22-Pad29) -> col_12
- U1 pad 4: row_3 -> col_3
- U1 pad 5: col_1 -> col_4
- U1 pad 6: col_2 -> col_5
- U1 pad 7: col_3 -> col_6
- U1 pad 9: col_4 -> row_1
Routing:
- net col_5: track 1.95 -> 103.1 mm, vias 0 -> 4
- net col_6: track 0.00 -> 95.0 mm, vias 0 -> 3
- net col_4: track 0.00 -> 78.4 mm, vias 0 -> 4
- net col_8: track 0.00 -> 77.7 mm, vias 0 -> 4
- net col_9: track 0.00 -> 74.7 mm, vias 0 -> 4
- net col_11: track 0.00 -> 49.5 mm, vias 0 -> 3
- net col_10: track 0.00 -> 45.6 mm, vias 0 -> 3
- net col_12: track 0.03 -> 45.4 mm, vias 0 -> 3
- net col_3: track 0.00 -> 44.6 mm, vias 0 -> 3
- net col_2: track 0.00 -> 44.3 mm, vias 0 -> 3

Commit message: few rows
Connections:
- U1 pad 1: col_1 -> col_6
- U1 pad 2: col_2 -> col_5
- U1 pad 22: col_7 -> col_12
- U1 pad 24: col_8 -> col_11
- U1 pad 25: col_9 -> col_10
- U1 pad 26: col_10 -> col_9
- U1 pad 27: col_11 -> col_8
- U1 pad 29: col_12 -> col_7
- U1 pad 4: col_3 -> col_4
- U1 pad 5: col_4 -> col_3
- U1 pad 6: col_5 -> col_2
- U1 pad 7: col_6 -> col_1
Routing:
- net col_4: track 78.4 -> 182.5 mm
- net col_5: track 103.1 -> 177.0 mm
- net col_6: track 95.0 -> 130.7 mm, vias 3 -> 4
Changed lines of the file:
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@@
 			(layers "*.Cu" "*.Mask")
 			(remove_unused_layers no)
-			(net 47 "col_1")
+			(net 52 "col_6")
 			(pinfunction "GPIO0")
 			(pintype "bidirectional")
@@
 			)
 			(layers "F.Cu" "F.Mask")
-			(net 47 "col_1")
+			(net 52 "col_6")
 			(pinfunction "GPIO0")
 			(pintype "bidirectional")
@@
 			(layers "*.Cu" "*.Mask")
 			(remove_unused_layers no)
-			(net 48 "col_2")
+			(net 51 "col_5")
 			(pinfunction "GPIO1")
 			(pintype "bidirectional")
@@
 			)
 			(layers "F.Cu" "F.Mask")
-			(net 48 "col_2")
+			(net 51 "col_5")
 			(pinfunction "GPIO1")
 			(pintype "bidirectional")
@@
 			(layers "*.Cu" "*.Mask")
 			(remove_unused_layers no)
-			(net 49 "col_3")
+			(net 50 "col_4")
 			(pinfunction "GPIO2")
 			(pintype "bidirectional")
@@
 			)
 			(layers "F.Cu" "F.Mask")
-			(net 49 "col_3")
+			(net 50 "col_4")
 			(pinfunction "GPIO2")
 			(pintype "bidirectional")
@@
 			(layers "*.Cu" "*.Mask")
 			(remove_unused_layers no)
-			(net 50 "col_4")
+			(net 49 "col_3")
 			(pinfunction "GPIO3")
 			(pintype "bidirectional")
@@
 			)
 			(layers "F.Cu" "F.Mask")
-			(net 50 "col_4")
+			(net 49 "col_3")
 			(pinfunction "GPIO3")
 			(pintype "bidirectional")
@@
 			(layers "*.Cu" "*.Mask")
 			(remove_unused_layers no)
-			(net 51 "col_5")
+			(net 48 "col_2")
 			(pinfunction "GPIO4")
 			(pintype "bidirectional")
@@
 			)
 			(layers "F.Cu" "F.Mask")
-			(net 51 "col_5")
+			(net 48 "col_2")
 			(pinfunction "GPIO4")
 			(pintype "bidirectional")
@@
 			(layers "*.Cu" "*.Mask")
 			(remove_unused_layers no)
-			(net 52 "col_6")
+			(net 47 "col_1")
 			(pinfunction "GPIO5")
 			(pintype "bidirectional")
@@
 			)
 			(layers "F.Cu" "F.Mask")
-			(net 52 "col_6")
+			(net 47 "col_1")
 			(pinfunction "GPIO5")
 			(pintype "bidirectional")
@@
 			(layers "*.Cu" "*.Mask")
 			(remove_unused_layers no)
-			(net 53 "col_7")
+			(net 58 "col_12")
 			(pinfunction "GPIO17")
 			(pintype "bidirectional")
@@
 			)
 			(layers "F.Cu" "F.Mask")
-			(net 53 "col_7")
+			(net 58 "col_12")
 			(pinfunction "GPIO17")
 			(pintype "bidirectional")
@@
 			(layers "*.Cu" "*.Mask")
 			(remove_unused_layers no)
-			(net 54 "col_8")
+			(net 57 "col_11")
 			(pinfunction "GPIO18")
 			(pintype "bidirectional")
@@
 			)
 			(layers "F.Cu" "F.Mask")
-			(net 54 "col_8")
+			(net 57 "col_11")
 			(pinfunction "GPIO18")
 			(pintype "bidirectional")
@@
 			(layers "*.Cu" "*.Mask")
 			(remove_unused_layers no)
-			(net 55 "col_9")
+			(net 56 "col_10")
 			(pinfunction "GPIO19")
 			(pintype "bidirectional")
@@
 			)
 			(layers "F.Cu" "F.Mask")
-			(net 55 "col_9")
+			(net 56 "col_10")
 			(pinfunction "GPIO19")
 			(pintype "bidirectional")
@@
 			(layers "*.Cu" "*.Mask")
 			(remove_unused_layers no)
-			(net 56 "col_10")
+			(net 55 "col_9")
 			(pinfunction "GPIO20")
 			(pintype "bidirectional")
@@
 			)
 			(layers "F.Cu" "F.Mask")
-			(net 56 "col_10")
+			(net 55 "col_9")
 			(pinfunction "GPIO20")
 			(pintype "bidirectional")
@@
 			(layers "*.Cu" "*.Mask")
 			(remove_unused_layers no)
-			(net 57 "col_11")
+			(net 54 "col_8")
 			(pinfunction "GPIO21")
 			(pintype "bidirectional")
@@
 			)
 			(layers "F.Cu" "F.Mask")
-			(net 57 "col_11")
+			(net 54 "col_8")
 			(pinfunction "GPIO21")
 			(pintype "bidirectional")
@@
 			(layers "*.Cu" "*.Mask")
 			(remove_unused_layers no)
-			(net 58 "col_12")
+			(net 53 "col_7")
 			(pinfunction "GPIO22")
 			(pintype "bidirectional")
@@
 			)
 			(layers "F.Cu" "F.Mask")
-			(net 58 "col_12")
+			(net 53 "col_7")
 			(pinfunction "GPIO22")
 			(pintype "bidirectional")
@@
 	)
 	(segment
+		(start 120.015 60.3885)
+		(end 109.1565 60.3885)
+		(width 0.2)
+		(layer "F.Cu")
+		(net 50)
+	)
+	(segment
+		(start 135.0645 68.58)
+		(end 128.2065 68.58)
+		(width 0.2)
+		(layer "F.Cu")
+		(net 50)
+	)
+	(segment
+		(start 109.1565 60.3885)
+		(end 103.632 54.864)
+		(width 0.2)
+		(layer "F.Cu")
+		(net 50)
+	)
+	(segment
 		(start 77.717442 92.467064)
 		(end 71.983815 108.220072)
@@
 	)
 	(segment
+		(start 140.2715 114.554)
+		(end 142.0495 114.554)
+		(width 0.2)
+		(layer "F.Cu")
+		(net 50)
+	)
+	(segment
 		(start 72.666955 109.68507)
 		(end 76.96323 111.248786)
@@
 	)
 	(segment
+		(start 103.632 54.864)
+		(end 93.346181 54.864)
+		(width 0.2)
+		(layer "F.Cu")
+		(net 50)
+	)
+	(segment
 		(start 90.292325 57.917856)
 		(end 77.717442 92.467064)
@@
 	)
 	(segment
+		(start 144.2085 77.724)
+		(end 135.0645 68.58)
+		(width 0.2)
+		(layer "F.Cu")
+		(net 50)
+	)
+	(segment
+		(start 144.2085 112.395)
+		(end 144.2085 77.724)
+		(width 0.2)
+		(layer "F.Cu")
+		(net 50)
+	)
+	(segment
+		(start 93.346181 54.864)
+		(end 90.292325 57.917856)
+		(width 0.2)
+		(layer "F.Cu")
+		(net 50)
+	)
+	(segment
 		(start 71.983815 108.220072)
 		(end 72.666955 109.68507)
@@
 		(net 50)
 	)
+	(segment
+		(start 128.2065 68.58)
+		(end 120.015 60.3885)
+		(width 0.2)
+		(layer "F.Cu")
+		(net 50)
+	)
+	(segment
+		(start 142.0495 114.554)
+		(end 144.2085 112.395)
+		(width 0.2)
+		(layer "F.Cu")
+		(net 50)
+	)
 	(via
 		(at 77.717442 92.467064)
@@
 	)
 	(segment
+		(start 142.875 108.585)
+		(end 142.875 78.105)
+		(width 0.2)
+		(layer "F.Cu")
+		(net 51)
+	)
+	(segment
 		(start 96.009514 97.90848)
 		(end 90.862282 112.050384)
@@
 	)
 	(segment
+		(start 119.492644 61.390144)
+		(end 109.301101 61.390144)
+		(width 0.2)
+		(layer "F.Cu")
+		(net 51)
+	)
+	(segment
 		(start 99.812197 117.537871)
 		(end 100.609193 119.247035)
@@
 	)
 	(segment
+		(start 141.986 109.474)
+		(end 142.875 108.585)
+		(width 0.2)
+		(layer "F.Cu")
+		(net 51)
+	)
+	(segment
+		(start 127.635 69.5325)
+		(end 119.492644 61.390144)
+		(width 0.2)
+		(layer "F.Cu")
+		(net 51)
+	)
+	(segment
 		(start 90.862282 112.050384)
 		(end 92.114705 114.736212)
@@
 	)
 	(segment
+		(start 142.875 78.105)
+		(end 134.3025 69.5325)
+		(width 0.2)
+		(layer "F.Cu")
+		(net 51)
+	)
+	(segment
 		(start 92.114705 114.736212)
 		(end 99.812197 117.537871)
@@
 	)
 	(segment
+		(start 134.3025 69.5325)
+		(end 127.635 69.5325)
+		(width 0.2)
+		(layer "F.Cu")
+		(net 51)
+	)
+	(segment
+		(start 140.2715 109.474)
+		(end 141.986 109.474)
+		(width 0.2)
+		(layer "F.Cu")
+		(net 51)
+	)
+	(segment
 		(start 109.301101 61.390144)
 		(end 96.009514 97.90848)
@@
 	)
 	(segment
-		(start 125.76884 71.84388)
+		(start 119.8245 88.2015)
 		(end 119.774594 88.312934)
 		(width 0.2)
@@
 	)
 	(segment
+		(start 115.23883 107.64617)
+		(end 115.951 106.934)
+		(width 0.2)
+		(layer "F.Cu")
+		(net 52)
+	)
+	(segment
+		(start 125.76884 71.84388)
+		(end 119.8245 88.2015)
+		(width 0.2)
+		(layer "F.Cu")
+		(net 52)
+	)
+	(segment
 		(start 113.584884 105.31902)
 		(end 112.737872 107.64617)
@@
 	)
 	(segment
+		(start 112.737872 107.64617)
+		(end 115.23883 107.64617)
+		(width 0.2)
+		(layer "F.Cu")
+		(net 52)
+	)
+	(segment
+		(start 115.951 106.934)
+		(end 140.2715 106.934)
+		(width 0.2)
+		(layer "F.Cu")
+		(net 52)
+	)
+	(segment
 		(start 119.20993 126.625328)
 		(end 120.120783 128.578657)
@@
 	)
 	(via
+		(at 119.8245 88.2015)
+		(size 0.6)
+		(drill 0.3)
+		(layers "F.Cu" "B.Cu")
+		(net 52)
+	)
+	(via
 		(at 112.737872 107.64617)
 		(size 0.6)
@@
 	)
 	(segment
+		(start 119.969243 94.910518)
+		(end 121.3485 93.531261)
+		(width 0.2)
+		(layer "B.Cu")
+		(net 52)
+	)
+	(segment
 		(start 114.195846 110.772802)
 		(end 112.737872 107.64617)
@@
 	)
 	(segment
+		(start 121.3485 89.7255)
+		(end 119.8245 88.2015)
+		(width 0.2)
+		(layer "B.Cu")
+		(net 52)
+	)
+	(segment
 		(start 113.453759 112.811664)
 		(end 114.195846 110.772802)
@@
 		(width 0.2)
 		(layer "B.Cu")
+		(net 52)
+	)
+	(segment
+		(start 121.3485 93.531261)
+		(end 121.3485 89.7255)
+		(width 0.2)
+		(layer "B.Cu")

Commit message: ergogen layout + elite-c
Parts:
- removed U1: Raspberry_Pi_Pico, ScottoKeebs_MCU:Raspberry_Pi_Pico
- added U2: Elite-C, Keebio-Parts:Elite-C, B.Cu at (149.2, 117.7)
- moved D38 7.49 mm to (111.5, 130.2)
- moved SW38 7.49 mm to (101.9, 128.7)
- moved D10 7.49 mm to (100.8, 77.3)
- moved D12 7.49 mm to (134.6, 95.7)
- moved D13 7.49 mm to (37.4, 84.4)
- moved D17 7.49 mm to (110.9, 105.3)
- moved D18 7.49 mm to (128.2, 113.4)
- moved D19 7.49 mm to (174.2, 71.9)
- moved D2 7.49 mm to (69.0, 53.3)
- moved D21 7.49 mm to (187.0, 107.2)
- moved D22 7.49 mm to (191.2, 63.1)
- moved D24 7.49 mm to (204.3, 98.9)
- moved D26 7.49 mm to (214.3, 70.9)
- moved D28 7.49 mm to (226.4, 48.3)
- moved D30 7.49 mm to (239.4, 84.1)
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Routing:
- net col_1: track 38.1 -> 168.8 mm, vias 0 -> 1
- net row_3: track 232.8 -> 354.4 mm, vias 0 -> 2
- net col_12: track 45.4 -> 164.9 mm, vias 3 -> 4
- net col_2: track 44.3 -> 154.3 mm
- net row_2: track 235.6 -> 341.2 mm, vias 0 -> 2
- net col_11: track 49.5 -> 146.8 mm
- net col_3: track 44.6 -> 133.7 mm
- net row_4: track 122.8 -> 211.5 mm
- net row_1: track 232.8 -> 317.5 mm, vias 0 -> 2
- net col_10: track 45.6 -> 121.3 mm, vias 3 -> 4
- net col_9: track 74.7 -> 117.2 mm
- net col_4: track 182.5 -> 143.0 mm
- net col_5: track 177.0 -> 141.6 mm
- net col_8: track 77.7 -> 100.4 mm
- net col_7: track 76.2 -> 95.8 mm
Other:
- board outline added: 268.6 x 131.4 mm
